File: Motor_Control/PCB_Design/MCB/V2/PCB_v2.sch (KiCad schematic (older format))
At the start: 26 parts, among them J1 Molex_Motor, J2 Conn_Encoder, J3 Molex_Pwr_In, J5 Molex_Pwr_Out, J6 Adress_Pins, J9 Conn_I2C, SW1 SW_DIP_x01, U1 DRV8308, U4 LM2931

Commit message: Footprint 2, tous ajoutés sauf les LED + Swtich
Parts:
- C1, C3, C4, C5, C6: footprint Capacitor_THT:C_Disc_D4.7mm_W2.5mm_P5.00mm -> Capacitor_SMD:C_1206_3216Metric_Pad1.42x1.75mm_HandSolder
- C2: footprint Capacitor_THT:CP_Radial_D8.0mm_P5.00mm -> Capacitor_SMD:CP_Elec_10x10
- R1, R2, R3, R4, R5: footprint Resistor_SMD:R_1206_3216Metric_Pad1.42x1.75mm_HandSolder -> Resistor_SMD:R_2010_5025Metric_Pad1.52x2.65mm_HandSolder
Changed lines of the file:
@@
 F 0 "C3" H 4315 2546 50  0000 L CNN
 F 1 "0.1uF" H 3900 2500 50  0000 L CNN
-F 2 "Capacitor_THT:C_Disc_D4.7mm_W2.5mm_P5.00mm" H 4238 2350 50  0001 C CNN
+F 2 "Capacitor_SMD:C_1206_3216Metric_Pad1.42x1.75mm_HandSolder" H 4238 2350 50  0001 C CNN
 F 3 "~" H 4200 2500 50  0001 C CNN
 	1    4200 2500
@@
 F 0 "C5" H 5200 1650 50  0000 L CNN
 F 1 "1uF" H 5350 1650 50  0000 L CNN
-F 2 "Capacitor_THT:C_Disc_D4.7mm_W2.5mm_P5.00mm" H 5338 1400 50  0001 C CNN
+F 2 "Capacitor_SMD:C_1206_3216Metric_Pad1.42x1.75mm_HandSolder" H 5338 1400 50  0001 C CNN
 F 3 "~" H 5300 1550 50  0001 C CNN
 	1    5300 1550
@@
 F 0 "C4" H 5050 2150 50  0000 L CNN
 F 1 "1uF" H 4750 2050 50  0000 L CNN
-F 2 "Capacitor_THT:C_Disc_D4.7mm_W2.5mm_P5.00mm" H 5038 1900 50  0001 C CNN
+F 2 "Capacitor_SMD:C_1206_3216Metric_Pad1.42x1.75mm_HandSolder" H 5038 1900 50  0001 C CNN
 F 3 "~" H 5000 2050 50  0001 C CNN
 	1    5000 2050
@@
 F 0 "C1" H 2600 1700 50  0000 C CNN
 F 1 "0.1uF" H 2500 1600 50  0000 C CNN
-F 2 "Capacitor_THT:C_Disc_D4.7mm_W2.5mm_P5.00mm" H 2738 1450 50  0001 C CNN
+F 2 "Capacitor_SMD:C_1206_3216Metric_Pad1.42x1.75mm_HandSolder" H 2738 1450 50  0001 C CNN
 F 3 "~" H 2700 1600 50  0001 C CNN
 	1    2700 1600
@@
 F 0 "C6" V 5648 1600 50  0000 C CNN
 F 1 "0.1uF" V 5739 1600 50  0000 C CNN
-F 2 "Capacitor_THT:C_Disc_D4.7mm_W2.5mm_P5.00mm" H 5938 1450 50  0001 C CNN
+F 2 "Capacitor_SMD:C_1206_3216Metric_Pad1.42x1.75mm_HandSolder" H 5938 1450 50  0001 C CNN
 F 3 "~" H 5900 1600 50  0001 C CNN
 	1    5900 1600
@@
 F 0 "R1" H 2170 4846 50  0000 L CNN
 F 1 "1K" H 2170 4755 50  0000 L CNN
-F 2 "Resistor_SMD:R_1206_3216Metric_Pad1.42x1.75mm_HandSolder" V 2030 4800 50  0001 C CNN
+F 2 "Resistor_SMD:R_2010_5025Metric_Pad1.52x2.65mm_HandSolder" V 2030 4800 50  0001 C CNN
 F 3 "~" H 2100 4800 50  0001 C CNN
 	1    2100 4800
@@
 F 0 "R2" H 2420 5246 50  0000 L CNN
 F 1 "1K" H 2420 5155 50  0000 L CNN
-F 2 "Resistor_SMD:R_1206_3216Metric_Pad1.42x1.75mm_HandSolder" V 2280 5200 50  0001 C CNN
+F 2 "Resistor_SMD:R_2010_5025Metric_Pad1.52x2.65mm_HandSolder" V 2280 5200 50  0001 C CNN
 F 3 "~" H 2350 5200 50  0001 C CNN
 	1    2350 5200
@@
 F 0 "R3" H 2670 5746 50  0000 L CNN
 F 1 "1K" H 2670 5655 50  0000 L CNN
-F 2 "Resistor_SMD:R_1206_3216Metric_Pad1.42x1.75mm_HandSolder" V 2530 5700 50  0001 C CNN
+F 2 "Resistor_SMD:R_2010_5025Metric_Pad1.52x2.65mm_HandSolder" V 2530 5700 50  0001 C CNN
 F 3 "~" H 2600 5700 50  0001 C CNN
 	1    2600 5700
@@
 F 0 "R4" H 3520 4896 50  0000 L CNN
 F 1 "1K" H 3520 4805 50  0000 L CNN
-F 2 "Resistor_SMD:R_1206_3216Metric_Pad1.42x1.75mm_HandSolder" V 3380 4850 50  0001 C CNN
+F 2 "Resistor_SMD:R_2010_5025Metric_Pad1.52x2.65mm_HandSolder" V 3380 4850 50  0001 C CNN
 F 3 "~" H 3450 4850 50  0001 C CNN
 	1    3450 4850
@@
 F 0 "R5" H 3520 5646 50  0000 L CNN
 F 1 "1K" H 3520 5555 50  0000 L CNN
-F 2 "Resistor_SMD:R_1206_3216Metric_Pad1.42x1.75mm_HandSolder" V 3380 5600 50  0001 C CNN
+F 2 "Resistor_SMD:R_2010_5025Metric_Pad1.52x2.65mm_HandSolder" V 3380 5600 50  0001 C CNN
 F 3 "~" H 3450 5600 50  0001 C CNN
 	1    3450 5600
@@
 F 0 "C2" H 3115 1646 50  0000 L CNN
 F 1 "470uF" H 3115 1555 50  0000 L CNN
-F 2 "Capacitor_THT:CP_Radial_D8.0mm_P5.00mm" H 3000 1600 50  0001 C CNN
+F 2 "Capacitor_SMD:CP_Elec_10x10" H 3000 1600 50  0001 C CNN
 F 3 "~" H 3000 1600 50  0001 C CNN
 	1    3000 1600

Commit message: Footprint des résistances pour les LEDS
Voir pour la PCB 1.5, car je crois que tout est prêt
Parts:
- 330ohm1, 330ohm2, 330ohm3: footprint (none) -> Resistor_SMD:R_2010_5025Metric_Pad1.52x2.65mm_HandSolder
- U4: symbol MyLibrary:LM2931 -> PCB_v2-rescue:LM2931-MyLibrary
Changed lines of the file:
@@
 F 0 "330ohm1" V 9993 5500 50  0000 C CNN
 F 1 "R10" V 10084 5500 50  0000 C CNN
-F 2 "" V 10130 5500 50  0001 C CNN
+F 2 "Resistor_SMD:R_2010_5025Metric_Pad1.52x2.65mm_HandSolder" V 10130 5500 50  0001 C CNN
 F 3 "~" H 10200 5500 50  0001 C CNN
 	1    10200 5500
@@
 F 0 "330ohm2" V 9993 5900 50  0000 C CNN
 F 1 "R11" V 10084 5900 50  0000 C CNN
-F 2 "" V 10130 5900 50  0001 C CNN
+F 2 "Resistor_SMD:R_2010_5025Metric_Pad1.52x2.65mm_HandSolder" V 10130 5900 50  0001 C CNN
 F 3 "~" H 10200 5900 50  0001 C CNN
 	1    10200 5900
@@
 F 0 "330ohm3" V 9993 6350 50  0000 C CNN
 F 1 "R13" V 10084 6350 50  0000 C CNN
-F 2 "" V 10130 6350 50  0001 C CNN
+F 2 "Resistor_SMD:R_2010_5025Metric_Pad1.52x2.65mm_HandSolder" V 10130 6350 50  0001 C CNN
 F 3 "~" H 10200 6350 50  0001 C CNN
 	1    10200 6350
@@
 LED3
 $Comp
-L MyLibrary:LM2931 U4
+L PCB_v2-rescue:LM2931-MyLibrary U4
 U 1 1 5DCAE5B5
 P 1350 1850
