File: Motor_Control/PCB_Design/MCB/V2/PCB_v2.sch (KiCad schematic (older format))
At the start: 26 parts, among them J1 Molex_Motor, J2 Conn_Encoder, J3 Molex_Pwr_In, J5 Molex_Pwr_Out, J6 Adress_Pins, J9 Conn_I2C, SW1 SW_DIP_x01, U1 DRV8308, U4 LM2931

Commit message: RIP LEDS
Parts:
- removed 330ohm1: R10, Resistor_SMD:R_2010_5025Metric_Pad1.52x2.65mm_HandSolder, symbol Device:R
- removed 330ohm2: R11, Resistor_SMD:R_2010_5025Metric_Pad1.52x2.65mm_HandSolder, symbol Device:R
- removed 330ohm3: R13, Resistor_SMD:R_2010_5025Metric_Pad1.52x2.65mm_HandSolder, symbol Device:R
- removed Rouge1: LED2, symbol Device:LED
- removed Rouge2: LED3, symbol Device:LED
- removed SW1: SW_DIP_x01, symbol Switch:SW_DIP_x01
- removed Vert1: LED1, symbol Device:LED
- J1: symbol PCB_v2-rescue:Molex_39-28-1083-MyLibrary -> PCB_v2-rescue:Molex_39-28-1083-MyLibrary-PCB_v2-rescue
Connections:
- net labels removed: Vm_in
- wire segments 179 -> 171
Other:
- note removed: "Connector of the LEDs"
Changed lines of the file:
@@
 EESchema Schematic File Version 4
 LIBS:PCB_v2-cache
-EELAYER 30 0
+EELAYER 26 0
 EELAYER END
 $Descr A4 11693 8268
@@
 $EndComp
 Text Label 2500 1400 0    50   ~ 0
-Vm_in
+Vm
 Wire Wire Line
 	3100 1350 3100 1400
@@
 Vreg
 $Comp
-L PCB_v2-rescue:Molex_39-28-1083-MyLibrary J1
+L PCB_v2-rescue:Molex_39-28-1083-MyLibrary-PCB_v2-rescue J1
 U 1 1 5BE0BE2F
 P 1750 3050
@@
 	1050 1300 1200 1300
 Text Label 1050 1200 2    50   ~ 0
-Vm_in
+Vm
 Wire Wire Line
 	1050 1200 1200 1200
@@
 	1100 800  1250 800
 Text Label 1100 700  2    50   ~ 0
-Vm_in
+Vm
 Wire Wire Line
 	1100 700  1250 700
@@
 	1050 1850 700  1850
 Text Label 700  1850 0    50   ~ 0
-Vm_in
+Vm
 Wire Wire Line
 	1650 1850 2000 1850
@@
 Wire Wire Line
 	10050 2650 10350 2650
-$Comp
-L Device:LED Vert1
-U 1 1 5DCA1693
-P 10500 5500
-F 0 "Vert1" H 10493 5245 50  0000 C CNN
-F 1 "LED1" H 10493 5336 50  0000 C CNN
-F 2 "" H 10500 5500 50  0001 C CNN
-F 3 "~" H 10500 5500 50  0001 C CNN
-	1    10500 5500
-	-1   0    0    1
-$EndComp
-$Comp
-L Device:LED Rouge1
-U 1 1 5DCB8BC5
-P 10500 5900
-F 0 "Rouge1" H 10493 5645 50  0000 C CNN
-F 1 "LED2" H 10493 5736 50  0000 C CNN
-F 2 "" H 10500 5900 50  0001 C CNN
-F 3 "~" H 10500 5900 50  0001 C CNN
-	1    10500 5900
-	-1   0    0    1
-$EndComp
-$Comp
-L Device:LED Rouge2
-U 1 1 5DCC2745
-P 10500 6350
-F 0 "Rouge2" H 10493 6095 50  0000 C CNN
-F 1 "LED3" H 10493 6186 50  0000 C CNN
-F 2 "" H 10500 6350 50  0001 C CNN
-F 3 "~" H 10500 6350 50  0001 C CNN
-	1    10500 6350
-	-1   0    0    1
-$EndComp
-Text Label 10800 5500 0    50   ~ 0
-GNDREF
 Text Label 10150 2450 0    50   ~ 0
 LED1
@@
 LED2
 Text Label 10150 2650 0    50   ~ 0
-LED3
-Wire Wire Line
-	10650 5500 11100 5500
-Wire Wire Line
-	10650 5900 11100 5900
-Wire Wire Line
-	10650 6350 11100 6350
-Text Label 10800 5900 0    50   ~ 0
-GNDREF
-Text Label 10800 6350 0    50   ~ 0
-GNDREF
-$Comp
-L Device:R 330ohm1
-U 1 1 5DDD767E
-P 10200 5500
-F 0 "330ohm1" V 9993 5500 50  0000 C CNN
-F 1 "R10" V 10084 5500 50  0000 C CNN
-F 2 "Resistor_SMD:R_2010_5025Metric_Pad1.52x2.65mm_HandSolder" V 10130 5500 50  0001 C CNN
-F 3 "~" H 10200 5500 50  0001 C CNN
-	1    10200 5500
-	0    1    1    0
-$EndComp
-$Comp
-L Device:R 330ohm2
-U 1 1 5DDF84A9
-P 10200 5900
-F 0 "330ohm2" V 9993 5900 50  0000 C CNN
-F 1 "R11" V 10084 5900 50  0000 C CNN
-F 2 "Resistor_SMD:R_2010_5025Metric_Pad1.52x2.65mm_HandSolder" V 10130 5900 50  0001 C CNN
-F 3 "~" H 10200 5900 50  0001 C CNN
-	1    10200 5900
-	0    1    1    0
-$EndComp
-$Comp
-L Device:R 330ohm3
-U 1 1 5DE026F6
-P 10200 6350
-F 0 "330ohm3" V 9993 6350 50  0000 C CNN
-F 1 "R13" V 10084 6350 50  0000 C CNN
-F 2 "Resistor_SMD:R_2010_5025Metric_Pad1.52x2.65mm_HandSolder" V 10130 6350 50  0001 C CNN
-F 3 "~" H 10200 6350 50  0001 C CNN
-	1    10200 6350
-	0    1    1    0
-$EndComp
-Wire Wire Line
-	10050 5500 9700 5500
-Wire Wire Line
-	10050 5900 9700 5900
-Wire Wire Line
-	10050 6350 9700 6350
-Text Notes 10000 5100 0    50   ~ 0
-Connector of the LEDs
-Text Label 9700 5500 0    50   ~ 0
-LED1
-Text Label 9700 5900 0    50   ~ 0
-LED2
-Text Label 9700 6350 0    50   ~ 0
 LED3
 $Comp
@@
 NoConn ~ 1200 1400
 NoConn ~ 1250 900
-$Comp
-L Switch:SW_DIP_x01 SW1
-U 1 1 5DCCF092
-P 2700 850
-F 0 "SW1" H 2700 1117 50  0000 C CNN
-F 1 "SW_DIP_x01" H 2700 1026 50  0000 C CNN
-F 2 "" H 2700 850 50  0001 C CNN
-F 3 "~" H 2700 850 50  0001 C CNN
-	1    2700 850
-	1    0    0    -1
-$EndComp
-Wire Wire Line
-	3000 850  3300 850
-Wire Wire Line
-	2400 850  2100 850
-Text Label 2100 850  0    50   ~ 0
-Vm_in
-Text Label 3200 850  0    50   ~ 0
-Vm
 Wire Wire Line
 	2550 3250 2800 3250

Commit message: PCB à jour, track manquante
Parts:
- J1: symbol PCB_v2-rescue:Molex_39-28-1083-MyLibrary-PCB_v2-rescue -> PCB_v2-rescue:Molex_39-28-1083-MyLibrary-PCB_v2-rescue-PCB_v2-rescue
- U4: symbol PCB_v2-rescue:LM2931-MyLibrary -> PCB_v2-rescue:LM2931-MyLibrary-PCB_v2-rescue
Changed lines of the file:
@@
 EESchema Schematic File Version 4
 LIBS:PCB_v2-cache
-EELAYER 26 0
+EELAYER 30 0
 EELAYER END
 $Descr A4 11693 8268
@@
 Vreg
 $Comp
-L PCB_v2-rescue:Molex_39-28-1083-MyLibrary-PCB_v2-rescue J1
+L PCB_v2-rescue:Molex_39-28-1083-MyLibrary-PCB_v2-rescue-PCB_v2-rescue J1
 U 1 1 5BE0BE2F
 P 1750 3050
@@
 LED3
 $Comp
-L PCB_v2-rescue:LM2931-MyLibrary U4
+L PCB_v2-rescue:LM2931-MyLibrary-PCB_v2-rescue U4
 U 1 1 5DCAE5B5
 P 1350 1850

Commit message: All routs
Parts:
- J1: symbol PCB_v2-rescue:Molex_39-28-1083-MyLibrary-PCB_v2-rescue-PCB_v2-rescue -> PCB_v2-rescue:Molex_39-28-1083-MyLibrary-PCB_v2-rescue-PCB_v2-rescue-PCB_v2-rescue
- U4: symbol PCB_v2-rescue:LM2931-MyLibrary-PCB_v2-rescue -> PCB_v2-rescue:LM2931-MyLibrary-PCB_v2-rescue-PCB_v2-rescue
Changed lines of the file:
@@
 EESchema Schematic File Version 4
 LIBS:PCB_v2-cache
-EELAYER 30 0
+EELAYER 26 0
 EELAYER END
 $Descr A4 11693 8268
@@
 Vreg
 $Comp
-L PCB_v2-rescue:Molex_39-28-1083-MyLibrary-PCB_v2-rescue-PCB_v2-rescue J1
+L PCB_v2-rescue:Molex_39-28-1083-MyLibrary-PCB_v2-rescue-PCB_v2-rescue-PCB_v2-rescue J1
 U 1 1 5BE0BE2F
 P 1750 3050
@@
 NoConn ~ 8600 5050
 Text Label 8900 5450 0    50   ~ 0
-Vreg
+Vin
 Text Label 8800 5250 0    50   ~ 0
 ENC_A
@@
 F4 "ENC_B" I L 4950 6450 50
 F5 "ENC_!B" I L 4950 6800 50
-F6 "Vreg" I R 6050 6250 50
+F6 "Vin" I R 6050 6250 50
 F7 "GND" I R 6050 6500 50
 F8 "3.3V" I R 6050 6750 50
@@
 	4600 6800 4950 6800
 Text Label 6400 6250 2    50   ~ 0
-Vreg
+Vin
 Wire Wire Line
 	6400 6250 6050 6250
@@
 LED3
 $Comp
-L PCB_v2-rescue:LM2931-MyLibrary-PCB_v2-rescue U4
+L PCB_v2-rescue:LM2931-MyLibrary-PCB_v2-rescue-PCB_v2-rescue U4
 U 1 1 5DCAE5B5
 P 1350 1850
