File: Motor_Control/PCB_Design/MCB/V2/PCB_v2.kicad_pcb (KiCad board)
At the start: 2 copper layers, 80.1 x 70 mm, 36 parts, among them J1 Molex_Motor, J2 Conn_Encoder, J3 Molex_Pwr_In, J4 Teensy, J5 Molex_Pwr_Out, J6 Adress_Pins, J9 Conn_I2C, Q1 Q_NMOS_IRLB8743, Q2 Q_NMOS_IRLB8743, Q3 Q_NMOS_IRLB8743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

Commit message: Fix du prob de ground
Routing:
- net GNDREF: track 55.9 -> 161.3 mm, vias 11 -> 14
- net /Vm: track 186.3 -> 185.8 mm
Changed lines of the file:
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@@
-(kicad_pcb (version 20171130) (host pcbnew "(5.0.0)")
+(kicad_pcb (version 20171130) (host pcbnew "(5.1.4)-1")
   (general
     (thickness 1.6)
     (drawings 14)
-    (tracks 524)
+    (tracks 546)
     (zones 0)
     (modules 36)
@@
     (0 F.Cu signal)
     (31 B.Cu signal)
-    (32 B.Adhes user)
-    (33 F.Adhes user)
+    (32 B.Adhes user hide)
+    (33 F.Adhes user hide)
     (34 B.Paste user)
     (35 F.Paste user)
-    (36 B.SilkS user)
-    (37 F.SilkS user)
-    (38 B.Mask user)
-    (39 F.Mask user)
+    (36 B.SilkS user hide)
+    (37 F.SilkS user hide)
+    (38 B.Mask user hide)
+    (39 F.Mask user hide)
     (40 Dwgs.User user)
     (41 Cmts.User user)
@@
     (47 F.CrtYd user)
     (48 B.Fab user)
-    (49 F.Fab user hide)
+    (49 F.Fab user)
   )
   (setup
-    (last_trace_width 1.5)
+    (last_trace_width 0.25)
     (user_trace_width 0.2)
     (user_trace_width 0.25)
@@
     (zone_45_only no)
     (trace_min 0.15)
-    (segment_width 0.2)
-    (edge_width 0.15)
     (via_size 0.8)
     (via_drill 0.4)
@@
     (uvia_min_size 0.2)
     (uvia_min_drill 0.1)
+    (edge_width 0.15)
+    (segment_width 0.2)
     (pcb_text_width 0.3)
     (pcb_text_size 1.5 1.5)
@@
   (via (at 127.5445 80.264) (size 0.8) (drill 0.4) (layers F.Cu B.Cu) (net 1))
   (via (at 127.073 95.758) (size 0.8) (drill 0.4) (layers F.Cu B.Cu) (net 1))
-  (segment (start 138.9898 113.03) (end 134.5702 108.6104) (width 1.5) (layer B.Cu) (net 1))
-  (segment (start 151.765 113.03) (end 138.9898 113.03) (width 1.5) (layer B.Cu) (net 1))
   (segment (start 135.89 87.63) (end 133.35 85.09) (width 1.5) (layer B.Cu) (net 1))
   (segment (start 151.765 87.63) (end 135.89 87.63) (width 1.5) (layer B.Cu) (net 1))
@@
   (segment (start 199.614999 121.695001) (end 199.614999 119.790001) (width 1.5) (layer B.Cu) (net 1))
   (segment (start 199.614999 119.790001) (end 202.565 116.84) (width 1.5) (layer B.Cu) (net 1))
-  (segment (start 127.635 116.205) (end 132.08 111.76) (width 1.5) (layer B.Cu) (net 1))
-  (segment (start 132.08 106.045) (end 131.445 105.41) (width 1.5) (layer B.Cu) (net 1))
-  (segment (start 132.08 111.76) (end 132.08 106.045) (width 1.5) (layer B.Cu) (net 1))
   (segment (start 134.62 108.585) (end 131.445 105.41) (width 1.5) (layer B.Cu) (net 1))
   (segment (start 131.445 105.41) (end 127 100.965) (width 1.5) (layer B.Cu) (net 1))
   (segment (start 130.81 104.775) (end 131.445 105.41) (width 1.5) (layer B.Cu) (net 1))
   (segment (start 130.81 103.505) (end 130.81 104.775) (width 1.5) (layer B.Cu) (net 1))
+  (segment (start 131.445 111.453416) (end 131.445 105.41) (width 1.5) (layer B.Cu) (net 1))
+  (segment (start 135.459984 108.6104) (end 134.5702 108.6104) (width 1.5) (layer B.Cu) (net 1))
+  (segment (start 127.635 116.205) (end 127.635 115.263416) (width 1.5) (layer B.Cu) (net 1))
+  (segment (start 139.879584 113.03) (end 135.459984 108.6104) (width 1.5) (layer B.Cu) (net 1))
+  (segment (start 127.635 115.263416) (end 131.445 111.453416) (width 1.5) (layer B.Cu) (net 1))
+  (segment (start 151.765 113.03) (end 139.879584 113.03) (width 1.5) (layer B.Cu) (net 1))
   (via (at 131.3688 95.7326) (size 0.8) (drill 0.4) (layers F.Cu B.Cu) (net 2))
   (segment (start 131.3434 95.758) (end 131.3688 95.7326) (width 0.15) (layer F.Cu) (net 2))
@@
   (segment (start 174.752 74.1075) (end 177.9875 74.1075) (width 1.5) (layer F.Cu) (net 2))
   (segment (start 177.9875 74.1075) (end 178.435 73.66) (width 1.5) (layer F.Cu) (net 2))
+  (segment (start 131.835 116.205) (end 131.835 112.512998) (width 0.15) (layer B.Cu) (net 2))
+  (segment (start 131.835 115.053) (end 132.08 114.808) (width 0.15) (layer B.Cu) (net 2))
+  (segment (start 131.835 116.205) (end 131.835 115.053) (width 0.15) (layer B.Cu) (net 2))
+  (segment (start 135.81 112.23) (end 135.81 103.505) (width 0.25) (layer F.Cu) (net 2))
+  (segment (start 131.835 116.205) (end 135.81 112.23) (width 0.25) (layer F.Cu) (net 2))
+  (segment (start 133.084999 117.454999) (end 134.726999 117.454999) (width 0.25) (layer F.Cu) (net 2))
+  (segment (start 131.835 116.205) (end 133.084999 117.454999) (width 0.25) (layer F.Cu) (net 2))
+  (segment (start 134.726999 117.454999) (end 143.764 126.492) (width 0.25) (layer F.Cu) (net 2))
+  (segment (start 143.764 126.492) (end 143.764 126.492) (width 0.25) (layer F.Cu) (net 2))
+  (via (at 143.764 126.492) (size 0.8) (drill 0.4) (layers F.Cu B.Cu) (net 2))
+  (segment (start 143.764 126.492) (end 143.764 126.492) (width 0.25) (layer F.Cu) (net 2))
+  (via (at 143.764 126.492) (size 0.8) (drill 0.4) (layers F.Cu B.Cu) (net 2))
+  (segment (start 143.764 126.492) (end 148.336 121.92) (width 0.25) (layer B.Cu) (net 2))
+  (segment (start 148.336 121.92) (end 148.844 122.428) (width 0.25) (layer B.Cu) (net 2))
+  (segment (start 148.844 122.428) (end 161.036 122.428) (width 0.25) (layer B.Cu) (net 2))
+  (segment (start 166.138012 127.530012) (end 197.589988 127.530012) (width 0.25) (layer B.Cu) (net 2))
+  (segment (start 161.036 122.428) (end 166.138012 127.530012) (width 0.25) (layer B.Cu) (net 2))
+  (segment (start 197.589988 127.530012) (end 197.589988 127.530012) (width 0.25) (layer B.Cu) (net 2))
+  (via (at 197.589988 127.530012) (size 0.8) (drill 0.4) (layers F.Cu B.Cu) (net 2))
+  (segment (start 197.589988 116.980012) (end 198.365 116.205) (width 0.25) (layer F.Cu) (net 2))
+  (segment (start 197.589988 127.530012) (end 197.589988 116.980012) (width 0.25) (layer F.Cu) (net 2))
   (segment (start 134.6565 78.130374) (end 136.320311 76.466563) (width 0.2) (layer F.Cu) (net 3))
   (segment (start 134.6565 80.264) (end 134.6565 78.130374) (width 0.2) (layer F.Cu) (net 3))
