File: Motor_Control/PCB_Design/MCB/V2/Power.sch (KiCad schematic (older format))
At the start: 7 parts, among them Q1 Q_NMOS_IRLB8743, Q2 Q_NMOS_IRLB8743, Q3 Q_NMOS_IRLB8743, Q4 Q_NMOS_IRLB8743, Q5 Q_NMOS_IRLB8743, Q6 Q_NMOS_IRLB8743

Commit message: Footprint 2, tous ajoutés sauf les LED + Swtich
Parts:
- R6: footprint Resistor_SMD:R_2512_6332Metric_Pad1.52x3.35mm_HandSolder -> Resistor_SMD:R_2010_5025Metric_Pad1.52x2.65mm_HandSolder
Changed lines of the file:
@@
 F 0 "R6" H 5220 4996 50  0000 L CNN
 F 1 "0.025" H 5220 4905 50  0000 L CNN
-F 2 "Resistor_SMD:R_2512_6332Metric_Pad1.52x3.35mm_HandSolder" V 5080 4950 50  0001 C CNN
+F 2 "Resistor_SMD:R_2010_5025Metric_Pad1.52x2.65mm_HandSolder" V 5080 4950 50  0001 C CNN
 F 3 "~" H 5150 4950 50  0001 C CNN
 	1    5150 4950
